File: Hardware/Production/Qwiic_Quad_Relay-Panel.brd (EAGLE design)
At the start: 179.3 x 123.7 mm, 483 parts, among them J10 Qwiic Right Angle, J11 Qwiic Right Angle, J12 AVR_SPI_PROG_3X2TESTPOINTS, J18 POWER_JACK, J19 Qwiic Right Angle, J2 Qwiic Right Angle, J20 Qwiic Right Angle, J21 AVR_SPI_PROG_3X2TESTPOINTS, J27 POWER_JACK, J28 Qwiic Right Angle, J29 Qwiic Right Angle, J3 Qwiic Right Angle, J30 AVR_SPI_PROG_3X2TESTPOINTS, J36 POWER_JACK, J4 AVR_SPI_PROG_3X2TESTPOINTS, J9 POWER_JACK, K1 RELAY-SPDT-JZC-11F, K10 RELAY-SPDT-JZC-11F, K11 RELAY-SPDT-JZC-11F, K12 RELAY-SPDT-JZC-11F, K13 RELAY-SPDT-JZC-11F, K14 RELAY-SPDT-JZC-11F, K15 RELAY-SPDT-JZC-11F, K16 RELAY-SPDT-JZC-11F, K2 RELAY-SPDT-JZC-11F, K3 RELAY-SPDT-JZC-11F, K4 RELAY-SPDT-JZC-11F, K5 RELAY-SPDT-JZC-11F, K6 RELAY-SPDT-JZC-11F, K7 RELAY-SPDT-JZC-11F, K8 RELAY-SPDT-JZC-11F, K9 RELAY-SPDT-JZC-11F, Q1 600mA/40V, Q10 600mA/40V, Q11 600mA/40V, Q12 600mA/40V, Q13 600mA/40V, Q14 600mA/40V, Q15 600mA/40V, Q16 600mA/40V, Q2 600mA/40V, Q3 600mA/40V, Q4 600mA/40V, Q5 600mA/40V, Q6 600mA/40V, Q7 600mA/40V, Q8 600mA/40V, Q9 600mA/40V, U10 DUAL-OPTOISOLATOR_SOIC8, U11 ATTINY84-ARDUINO, U13 DUAL-OPTOISOLATOR_SOIC8, U14 DUAL-OPTOISOLATOR_SOIC8, U15 ATTINY84-ARDUINO, U2 DUAL-OPTOISOLATOR_SOIC8, U3 DUAL-OPTOISOLATOR_SOIC8, U4 DUAL-OPTOISOLATOR_SOIC8, U5 ATTINY84-ARDUINO, U6 DUAL-OPTOISOLATOR_SOIC8, U7 ATTINY84-ARDUINO, U9 DUAL-OPTOISOLATOR_SOIC8

Commit message: panel
Parts:
- removed U$213, U$220: (no value), Labels:SCK-[)-03
- removed U$214, U$217: (no value), Labels:GND-03
- removed U$215, U$218: (no value), 5V:5V0
- removed U$216, U$219: (no value), SDA:SDA0
- removed U$221, U$223: (no value), Polarity_marking_center_positive#jpg:POLARITY_MARKING_CENTER_POSITIVE#JPG
- removed U$222: (no value), 7-15V:7#15V0
- removed U$224, U$225: (no value), qwiic_copyrighted_logo_medium:QWIIC#JPG
- removed U$226: (no value), 5V Wall Adapter:5V_WALL_ADAPTER0
- removed U$227: (no value), jumper:JUMPER0
- removed U$228: (no value), Labels:ADR-()-04
- added LOGO10, LOGO7: OSHW-LOGOS, SparkFun-Aesthetics:OSHW-LOGO-S
- added LOGO11, LOGO12, LOGO5, LOGO6, LOGO8, LOGO9: SFE_LOGO_NAME_FLAME.1_INCH, SparkFun-Aesthetics:SFE_LOGO_NAME_FLAME_.1
- D12, D2, D22, D32: value WHITE -> BLUE
- D18, D28, D38, D8: value Yellow -> BLUE
- D19, D29, D39, D9: value GREEN -> BLUE
- LOGO2, LOGO3: value OSHW-LOGOS -> SFE_LOGO_NAME_FLAME.1_INCH; device SparkFun-Aesthetics:OSHW-LOGO-S -> SparkFun-Aesthetics:SFE_LOGO_NAME_FLAME_.1
- R1, R12, R13, R14, R18, R27, R28, R29, R35, R44, R45, R46, R52, R61, R62, R63: value 10 -> 33
- R10, R11, R2, R23, R24, R25, R26, R3, R40, R41, R42, R43, R57, R58, R59, R60: value 220 -> 100
- R20, R37, R5, R54: value 220 -> 330
- U$10, U$158: device 5V:5V0 -> Labels:3V3-03
- U$100: device Labels:GND-03 -> 7-15V:7#15V0
- U$101: device 5V:5V0 -> Polarity_marking_center_positive#jpg:POLARITY_MARKING_CENTER_POSITIVE#JPG
- U$102: device SDA:SDA0 -> 5V Wall Adapter:5V_WALL_ADAPTER0
- U$103: device Labels:GND-03 -> jumper:JUMPER0
- U$104: device 5V:5V0 -> Labels:ADR-()-04
- U$105, U$159: device SDA:SDA0 -> Labels:3V3-03
- U$106: device Labels:SCK-[)-03 -> Labels:3V3-03
- U$107: device Polarity_marking_center_positive#jpg:POLARITY_MARKING_CENTER_POSITIVE#JPG -> Labels:PWR-()-04
- U$108: device 7-15V:7#15V0 -> 2:20
- U$109: device Polarity_marking_center_positive#jpg:POLARITY_MARKING_CENTER_POSITIVE#JPG -> 1:10
- U$110, U$57: device qwiic_copyrighted_logo_medium:QWIIC#JPG -> 3:30
- U$111: device qwiic_copyrighted_logo_medium:QWIIC#JPG -> 4:40
- U$112: device 5V Wall Adapter:5V_WALL_ADAPTER0 -> Quad:QWIIC_QUAD_0
- U$113: device jumper:JUMPER0 -> relay:RELAY0
- U$114: device Labels:ADR-()-04 -> NO:NO0
- U$115: device Labels:PWR-()-04 -> COM:COM0
- U$116: device 2:20 -> NC:NC0
- U$117: device 1:10 -> NO:NO0
- U$118: device 3:30 -> COM:COM0
- U$119: device 4:40 -> NC:NC0
- U$12: value SPARKX-LOGO4 -> (none); device SparkX:SPARKX-MEDIUM -> Labels:3V3-03
- U$120: device Quad:QWIIC_QUAD_0 -> NO:NO0
- U$121: device relay:RELAY0 -> COM:COM0
- U$122: value SPARKX-LOGO4 -> (none); device SparkX:SPARKX-MEDIUM -> NC:NC0
- U$123: device SparkX:SPARKX-MEDIUM -> NO:NO0
- U$124, U$127, U$130, U$133, U$136: device NO:NO0 -> COM:COM0
- U$125, U$128, U$131, U$134, U$137: device COM:COM0 -> NC:NC0
- U$126, U$129, U$132, U$135: device NC:NC0 -> NO:NO0
- U$138: device NC:NC0 -> 1:10
- U$139: device NO:NO0 -> 2:20
- U$14: device SparkX:SPARKX-MEDIUM -> Labels:PWR-()-04
- U$140: device COM:COM0 -> 3:30
- U$141: device NC:NC0 -> 4:40
- U$142: device NO:NO0 -> Quad:QWIIC_QUAD_0
- U$143: device COM:COM0 -> relay:RELAY0
- U$144: device NC:NC0 -> SparkFun-Aesthetics:OSHW-LOGO-S
- U$145: device NO:NO0 -> 7-15V:7#15V0
- U$146: device COM:COM0 -> Labels:SCK-[)-03
- U$147: device NC:NC0 -> Labels:GND-03
- U$148: device 1:10 -> SDA:SDA0
- U$149: device 2:20 -> Labels:GND-03
- U$150: device 3:30 -> SDA:SDA0
- U$151: device 4:40 -> Labels:SCK-[)-03
- U$152: device Quad:QWIIC_QUAD_0 -> Polarity_marking_center_positive#jpg:POLARITY_MARKING_CENTER_POSITIVE#JPG
- U$153: device relay:RELAY0 -> 7-15V:7#15V0
- U$154: device SparkFun-Aesthetics:OSHW-LOGO-S -> Polarity_marking_center_positive#jpg:POLARITY_MARKING_CENTER_POSITIVE#JPG
- U$155: device 7-15V:7#15V0 -> 5V Wall Adapter:5V_WALL_ADAPTER0
- U$156: device Labels:SCK-[)-03 -> jumper:JUMPER0
- U$157: device Labels:GND-03 -> Labels:ADR-()-04
- U$160: device Labels:GND-03 -> Labels:PWR-()-04
- U$161, U$46: device 5V:5V0 -> 2:20
- U$162: device SDA:SDA0 -> 1:10
- U$163: device Labels:SCK-[)-03 -> 3:30
- U$164: device Polarity_marking_center_positive#jpg:POLARITY_MARKING_CENTER_POSITIVE#JPG -> 4:40
- U$165: device 7-15V:7#15V0 -> Quad:QWIIC_QUAD_0
- U$166: device Polarity_marking_center_positive#jpg:POLARITY_MARKING_CENTER_POSITIVE#JPG -> relay:RELAY0
- U$167: device qwiic_copyrighted_logo_medium:QWIIC#JPG -> NO:NO0
- U$168: device qwiic_copyrighted_logo_medium:QWIIC#JPG -> COM:COM0
- U$169: device 5V Wall Adapter:5V_WALL_ADAPTER0 -> NC:NC0
- U$170: device jumper:JUMPER0 -> NO:NO0
- U$171: device Labels:ADR-()-04 -> COM:COM0
- U$172: device Labels:PWR-()-04 -> NC:NC0
- U$173: device 2:20 -> NO:NO0
- U$174: device 1:10 -> COM:COM0
- U$175: device 3:30 -> NC:NC0
- U$176: device 4:40 -> NO:NO0
- U$177: device Quad:QWIIC_QUAD_0 -> COM:COM0
- U$178: device relay:RELAY0 -> NC:NC0
- U$179: value SPARKX-LOGO4 -> (none); device SparkX:SPARKX-MEDIUM -> NO:NO0
- U$180: device SparkX:SPARKX-MEDIUM -> COM:COM0
- U$181, U$184, U$187, U$190: device NO:NO0 -> NC:NC0
- U$182, U$185, U$188: device COM:COM0 -> NO:NO0
- U$183, U$186, U$189: device NC:NC0 -> COM:COM0
- U$191: device COM:COM0 -> 1:10
- U$192: device NC:NC0 -> 2:20
- U$193: device NO:NO0 -> 3:30
- U$194: device COM:COM0 -> 4:40
- U$195: device NC:NC0 -> Quad:QWIIC_QUAD_0
- U$196: device NO:NO0 -> relay:RELAY0
- U$197: device COM:COM0 -> SparkFun-Aesthetics:OSHW-LOGO-S
- U$198: device NC:NC0 -> 7-15V:7#15V0
- U$199: device NO:NO0 -> Labels:SCK-[)-03
- U$200: device COM:COM0 -> Labels:GND-03
- U$201: device NC:NC0 -> SDA:SDA0
- U$202: device NO:NO0 -> Labels:GND-03
- U$203: device COM:COM0 -> SDA:SDA0
- U$204: device NC:NC0 -> Labels:SCK-[)-03
- U$205: device 1:10 -> Polarity_marking_center_positive#jpg:POLARITY_MARKING_CENTER_POSITIVE#JPG
- U$206, U$92: device 2:20 -> 7-15V:7#15V0
- U$207: device 3:30 -> Polarity_marking_center_positive#jpg:POLARITY_MARKING_CENTER_POSITIVE#JPG
- U$208: device 4:40 -> 5V Wall Adapter:5V_WALL_ADAPTER0
- U$209: device Quad:QWIIC_QUAD_0 -> jumper:JUMPER0
- U$210: device relay:RELAY0 -> Labels:ADR-()-04
- U$211: device SparkFun-Aesthetics:OSHW-LOGO-S -> Labels:3V3-03
- U$212: device 7-15V:7#15V0 -> Labels:3V3-03
- U$55: device qwiic_copyrighted_logo_medium:QWIIC#JPG -> 1:10
- U$58: device Labels:PWR-()-04 -> 4:40
- U$59: device 2:20 -> Quad:QWIIC_QUAD_0
- U$60: device 1:10 -> relay:RELAY0
- U$61: device 3:30 -> NO:NO0
- U$62: device 4:40 -> COM:COM0
- U$63: device Quad:QWIIC_QUAD_0 -> NC:NC0
- U$64: device relay:RELAY0 -> NO:NO0
- U$65: value SPARKX-LOGO4 -> (none); device SparkX:SPARKX-MEDIUM -> COM:COM0
- U$66: device SparkX:SPARKX-MEDIUM -> NC:NC0
- U$85: device NO:NO0 -> 1:10
- U$86: device COM:COM0 -> 2:20
- U$87: device NC:NC0 -> 3:30
- U$88: device NO:NO0 -> 4:40
- U$89: device COM:COM0 -> Quad:QWIIC_QUAD_0
- U$90: device NC:NC0 -> relay:RELAY0
- U$91: device 1:10 -> SparkFun-Aesthetics:OSHW-LOGO-S
- U$93: device 3:30 -> Labels:SCK-[)-03
- U$94: device 4:40 -> Labels:GND-03
- U$95: device Quad:QWIIC_QUAD_0 -> SDA:SDA0
- U$96: device relay:RELAY0 -> Labels:GND-03
- U$97: device SparkFun-Aesthetics:OSHW-LOGO-S -> SDA:SDA0
- U$98: device 7-15V:7#15V0 -> Labels:SCK-[)-03
- U$99: device Labels:SCK-[)-03 -> Polarity_marking_center_positive#jpg:POLARITY_MARKING_CENTER_POSITIVE#JPG
- moved U$195 186.7 mm to (28.3, 194.6), turned to 0 degrees
- moved U$196 184.6 mm to (18.0, 191.5), turned to 0 degrees
- moved U$112 182.8 mm to (3.81, 144.5), flipped to the top
- moved U$197 179.9 mm to (2.16, 180.3), turned to 0 degrees
- moved U$113 179.0 mm to (4.19, 141.5), flipped to the top
- moved U$191 178.8 mm to (19.3, 179.3), flipped to the bottom, turned to 0 degrees
- moved U$109 169.3 mm to (6.35, 129.3), flipped to the top
- moved U$192 168.4 mm to (38.9, 179.3), flipped to the bottom, turned to 0 degrees
- moved U$200 164.6 mm to (27.9, 195.5), flipped to the top
- moved U$201 164.4 mm to (33.0, 195.5), flipped to the top
- moved U$212 163.0 mm to (30.5, 195.5), flipped to the bottom
- moved U$108 158.3 mm to (25.4, 129.3), flipped to the top, turned to 0 degrees
- moved U$199 158.0 mm to (35.6, 195.5), flipped to the top
- moved U$190 157.9 mm to (21.6, 156.2), flipped to the bottom
- moved U$188 156.9 mm to (11.7, 156.3), flipped to the bottom
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Connections:
- net 3.3V: now also C1.1, J1.3, J4.2, R8.1, U5.1
- net 3.3V1: now also C5.1, J12.2, J14.3, R21.1, U7.1
- net 3.3V2: now also C9.1, J21.2, J23.3, R38.1, U11.1
- net 3.3V3: now also C13.1, J30.2, J32.3, R55.1, U15.1
- net 5V: no longer C1.1, J1.3, J4.2, R8.1, U5.1
- net 5V1: no longer C5.1, J12.2, J14.3, R21.1, U7.1
- net 5V2: no longer C9.1, J21.2, J23.3, R38.1, U11.1
- net 5V3: no longer C13.1, J30.2, J32.3, R55.1, U15.1
Routing:
- net 5V2: track 146.4 -> 121.6 mm, vias 6 -> 11
- net 5V1: track 146.4 -> 121.6 mm, vias 6 -> 11
- net 5V: track 146.4 -> 121.6 mm, vias 6 -> 11
- net 5V3: track 146.4 -> 121.6 mm, vias 6 -> 11
- net 3.3V1: track 82.9 -> 101.2 mm, vias 2 -> 4
- net 3.3V3: track 82.9 -> 101.2 mm, vias 2 -> 4
- net 3.3V: track 82.9 -> 101.2 mm, vias 2 -> 4
- net 3.3V2: track 82.9 -> 101.2 mm, vias 2 -> 4
- net SDA/MOSI2: track 112.0 -> 111.1 mm
- net SDA/MOSI3: track 112.0 -> 111.1 mm
- net SDA/MOSI: track 112.0 -> 111.1 mm
- net SDA/MOSI1: track 112.0 -> 111.1 mm
Other:
- board size 179.3 x 123.7 mm -> 96.3 x 222.2 mm
- board text added: "v10"
- board text removed: "x02"
